Commit message: update moveit and add gripper urdf

File: urdf/mycobot_urdf.urdf (robot description, URDF)
Before this commit: robot firefighter, 7 links, 6 joints
Links:
- added link gripper; collision mesh filename=package://mycobot_ros/urdf/gripper_ag.dae; visual mesh filename=package://mycobot_ros/urdf/gripper_ag.dae
Joints:
- added joint gitpper_to_joint6output: type fixed, parent joint6_flange, child gripper, origin xyz=0 0 0 rpy=0 0 0 , axis 0 0 1, limit lower=-3.14 upper=3.14159 effort=1000.0 velocity=0
