Commit message: update urdf

File: urdf/mycobot/mycobot_urdf.urdf (robot description, URDF)
Before this commit: robot firefighter, 8 links, 7 joints
Links:
- link gripper: geometry collision mesh filename=package://mycobot_ros/urdf/mycobot/gripper_ag.dae; visual mesh filename=package://mycobot_ros/urdf/mycobot/gripper_ag.dae
- link joint1: geometry collision mesh filename=package://mycobot_ros/urdf/mycobot/joint1.dae; visual mesh filename=package://mycobot_ros/urdf/mycobot/joint1.dae
- link joint2: geometry collision mesh filename=package://mycobot_ros/urdf/mycobot/joint2.dae; visual mesh filename=package://mycobot_ros/urdf/mycobot/joint2.dae
- link joint3: geometry collision mesh filename=package://mycobot_ros/urdf/mycobot/joint3.dae; visual mesh filename=package://mycobot_ros/urdf/mycobot/joint3.dae
- link joint4: geometry collision mesh filename=package://mycobot_ros/urdf/mycobot/joint4.dae; visual mesh filename=package://mycobot_ros/urdf/mycobot/joint4.dae
- link joint5: geometry collision mesh filename=package://mycobot_ros/urdf/mycobot/joint5.dae; visual mesh filename=package://mycobot_ros/urdf/mycobot/joint5.dae
- link joint6: geometry collision mesh filename=package://mycobot_ros/urdf/mycobot/joint6.dae; visual mesh filename=package://mycobot_ros/urdf/mycobot/joint6.dae
- link joint6_flange: geometry collision mesh filename=package://mycobot_ros/urdf/mycobot/joint7.dae; visual mesh filename=package://mycobot_ros/urdf/mycobot/joint7.dae

Commit message: fix typo

File: urdf/mycobot/mycobot_urdf.urdf (robot description, URDF)
Before this commit: robot firefighter, 8 links, 7 joints
Joints:
- removed joint gitpper_to_joint6output
- added joint gripper_to_joint6output: type fixed, parent joint6_flange, child gripper, origin xyz=0 0 0 rpy=0 0 0 , axis 0 0 1, limit lower=-3.14 upper=3.14159 effort=1000.0 velocity=0
