Commit message: update mycobot urdf

File: urdf/mycobot/mycobot_macro.xacro (robot description, xacro)
@@ -172,5 +172,5 @@
         <parent link="${prefix}joint6_flange"/>
         <child link="${prefix}gripper"/>
-        <origin xyz= "0 0 0" rpy = "0 0 0 "/>
+        <origin xyz= "0 0 0" rpy = "0 0 1 "/>
     </joint>
     </xacro:macro>

File: urdf/mycobot/mycobot_urdf.urdf (robot description, URDF)
Before this commit: robot firefighter, 8 links, 7 joints
Joints:
- joint gripper_to_joint6output: origin xyz=0 0 0 rpy=0 0 0  -> xyz=0 0 0 rpy=0 0 1 
